Commit message: Updated torso

File: urdf/quori_v2.urdf (robot description, URDF)
Before this commit: robot quori, 10 links, 9 joints
Links:
- link upper_torso: geometry visual mesh filename=package://quori_description/meshes/181010_Upper Torso Vente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

Commit message: repositioned a few joints and aligned the meshes better. Added camera and microphone frame

File: urdf/quori_v2.urdf (robot description, URDF)
Before this commit: robot quori, 10 links, 9 joints
Links:
- added link head_camera; visual box size=0.04 0.11 0.04
- added link head_mic; visual cylinder length=0.002 radius=0.03
- added link left_arm_upper2lower; visual cylinder length=0.08 radius=0.015
- added link right_arm_upper2lower; visual cylinder length=0.08 radius=0.015
- link upper_torso: geometry visual mesh filename=package://quori_description/meshes/0917_Upper Torso+Waist.d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
Joints:
- added joint head_Camera_joint: type fixed, parent head, child head_camera, origin xyz=0.055 0 0.21 rpy=0 0 0
- added joint head_Mic_joint: type fixed, parent head, child head_mic, origin xyz=-0.008 0 0.218 rpy=0 -.3 0
- added joint left_arm_upper2lower_j: type fixed, parent left_arm_upper, child left_arm_upper2lower
- added joint right_arm_upper2lower_j: type fixed, parent right_arm_upper, child right_arm_upper2lower
- joint head_joint: origin xyz=0 0 0 rpy=0 0 0 -> xyz=0 0 0.554 rpy=0 0 0
- joint left_arm_lower_r1: origin xyz=0 0 0 rpy=0 0 0 -> xyz=0 0.15 0 rpy=0 0 0
- joint left_arm_r2: axis 1 0 0 -> 0 0 1
- joint right_arm_lower_r1: origin xyz=0 0 0 rpy=0 0 0 -> xyz=0 -0.15 0 rpy=0 0 0
- joint right_arm_r2: axis 1 0 0 -> 0 0 1
