Commit message: canonicalize names

File: urdf/quori.urdf (robot description, URDF)
Before this commit: robot quori, 7 links, 6 joints
Links:
- link left_arm_upper: geometry visual mesh filename=package://quori_description/meshes/Left Arm.dae
- link lower_torso: geometry visual mesh filename=package://quori_description/meshes/Lower Torso.dae
- link right_arm_upper: geometry visual mesh filename=package://quori_description/meshes/Right Arm.dae
- link upper_torso: geometry visual mesh filename=package://quori_description/meshes/Upper Torso.dae

Commit message: updateing urdf file as it did not get pushed last time.

File: urdf/quori.urdf (robot description, URDF)
Before this commit: robot quori, 7 links, 6 joints
Links:
- added link head; visual mesh filename=package://quori_description/meshes/0917_Helmet_Duripod.dae
- added link head_camera; visual box size=0.04 0.11 0.04
- added link head_mic; visual cylinder length=0.002 radius=0.03
- added link left_arm_lower; visual mesh filename=package://quori_description/meshes/0917_Lower_Arm_left.dae
- added link left_arm_upper2lower; visual cylinder length=0.08 radius=0.015
- added link right_arm_lower; visual mesh filename=package://quori_description/meshes/0917_Lower Arm_right.dae
- added link right_arm_upper2lower; visual cylinder length=0.08 radius=0.015
- link left_arm_upper: geometry visual mesh filename=package://quori_description/meshes/0917_Upper Arm+gear_left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
- link lower_torso: geometry visual mesh filename=package://quori_description/meshes/180915_Lower Torso.dae
- link right_arm_upper: geometry visual mesh filename=package://quori_description/meshes/0917_Upper Arm+gear_righ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
- link upper_torso: geometry visual mesh filename=package://quori_description/meshes/0917_Upper Torso+Waist.d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
Joints:
- added joint head_Camera_joint: type fixed, parent head, child head_camera, origin xyz=0.055 0 0.21 rpy=0 0 0
- added joint head_Mic_joint: type fixed, parent head, child head_mic, origin xyz=-0.008 0 0.218 rpy=0 -.3 0
- added joint head_joint: type fixed, parent upper_torso, child head, origin xyz=0 0 0.554 rpy=0 0 0
- added joint left_arm_lower_r1: type revolute, parent left_arm_upper, child left_arm_lower, origin xyz=0 0.15 0 rpy=0 0 0, axis 0 1 0, limit lower=-1.1 upper=1.1 effort=1 velocity=3
- added joint left_arm_upper2lower_j: type fixed, parent left_arm_upper, child left_arm_upper2lower
- added joint right_arm_lower_r1: type revolute, parent right_arm_upper, child right_arm_lower, origin xyz=0 -0.15 0 rpy=0 0 0, axis 0 1 0, limit lower=-3.14 upper=3.14 effort=1 velocity=3
- added joint right_arm_upper2lower_j: type fixed, parent right_arm_upper, child right_arm_upper2lower
- joint left_arm_r2: axis 1 0 0 -> 0 0 1
- joint right_arm_r2: axis 1 0 0 -> 0 0 1

Commit message: updated the arm frames so the position control matches the robot hardware. updated the joint types and limits. added a place holder for the laser scanner.

File: urdf/quori.urdf (robot description, URDF)
Before this commit: robot quori, 14 links, 13 joints
Links:
- added link base_laser_scanner; visual cylinder length=0.025 radius=0.05
Joints:
- added joint laser_scanner_joint: type fixed, parent base_link, child base_laser_scanner, origin xyz=0.178 0 0.1 rpy=0 0 0
- joint left_arm_lower_r1: limit lower=-1.1 upper=1.1 effort=1 velocity=3 -> lower=-3.142 upper=3.142 effort=1 velocity=1; origin xyz=0 0.15 0 rpy=0 0 0 -> xyz=0 0.15 0 rpy=0 1.57 0
- joint left_arm_r1: limit lower=-3.14 upper=3.14 effort=1 velocity=3 -> effort=1 velocity=1; type revolute -> continuous
- joint left_arm_r2: axis 0 0 1 -> 0 0 -1; limit lower=-1.1 upper=1.1 effort=1 velocity=3 -> lower=-1.1 upper=1.1 effort=1 velocity=1; origin xyz=0 0 0 rpy=0 0 0 -> xyz=0 0 0 rpy=0 -1.57 0
- joint right_arm_lower_r1: limit lower=-3.14 upper=3.14 effort=1 velocity=3 -> lower=-3.14 upper=3.14 effort=1 velocity=1; origin xyz=0 -0.15 0 rpy=0 0 0 -> xyz=0 -0.15 0 rpy=0 1.57 0
- joint right_arm_r1: axis 0 1 0 -> 0 -1 0; limit lower=-3.14 upper=3.14 effort=1 velocity=3 -> effort=1 velocity=1; type revolute -> continuous
- joint right_arm_r2: limit lower=-1.1 upper=1.1 effort=1 velocity=3 -> lower=-1.1 upper=1.1 effort=1 velocity=1; origin xyz=0 0 0 rpy=0 0 0 -> xyz=0 0 0 rpy=0 -1.57 0
- joint turret_joint: limit lower=-3.14 upper=3.14 effort=1 velocity=3 -> effort=1 velocity=3; type revolute -> continuous
- joint waist_hinge: limit lower=-0.26 upper=0.52 effort=1 velocity=3 -> lower=-0.21 upper=0.47 effort=1 velocity=1

Commit message: adding inertial tags with nominal values. Update of values may be needed pending testing. files compile in RViz.

File: urdf/quori.urdf (robot description, URDF)
Before this commit: robot quori, 15 links, 14 joints
Links:
- link base_laser_scanner: mass None -> 0.17
- link base_link: mass None -> 9.8
- link head: mass None -> 1.9
- link head_camera: mass None -> 0.3
- link head_mic: mass None -> 0.05
- link left_arm_base: mass None -> 0.0
- link left_arm_lower: mass None -> 0.00
- link left_arm_upper: mass None -> 0.00
- link left_arm_upper2lower: mass None -> 0.19
- link lower_torso: mass None -> 2
- link right_arm_base: mass None -> 0.0
- link right_arm_lower: mass None -> 0.00
- link right_arm_upper: mass None -> 0.00
- link right_arm_upper2lower: mass None -> 0.19
- link upper_torso: mass None -> 26.75
